Commit message: My changes

File: src/hockey_robot_description/urdf/hockey_robot.urdf.xacro (robot description, xacro)
@@ -6,4 +6,6 @@
   <xacro:arg name="prefix" default=""/>
   <xacro:property name="prefix" value="$(arg prefix)"/>
+  <xacro:arg name="ns" default=""/>
+  <xacro:property name="ns" value="$(arg ns)"/>
   <!-- ========================= -->
   <!-- Dimensions -->
@@ -43,4 +45,5 @@
         <box size="${base_length} ${base_width} ${base_height}"/>
       </geometry>
+      <origin xyz=" 0 0 0.02" rpy = "0 0 0"/>
       <material name="Blue"/>
     </visual>
@@ -49,4 +52,5 @@
         <box size="${base_length} ${base_width} ${base_height}"/>
       </geometry>
+      <origin xyz=" 0 0 0.02" rpy = "0 0 0"/>
     </collision>
     <inertial>
@@ -65,12 +69,12 @@
         <cylinder radius="${wheel_radius}" length="${wheel_width}"/>
       </geometry>
-      <origin rpy="0 1.5708 0"/>
+      <origin rpy="-1.5708 0 0"/>
       <material name="Black"/>
     </visual>
     <collision>
       <geometry>
-        <cylinder radius="${wheel_radius}" length="${wheel_width}"/>
-      </geometry>
-      <origin rpy="0 1.5708 0"/>
+        <sphere radius="${wheel_radius}"/>
+      </geometry>
+      <origin rpy="-1.5708 0 0"/>
     </collision>
     <inertial>
@@ -94,10 +98,10 @@
         <cylinder radius="${wheel_radius}" length="${wheel_width}"/>
       </geometry>
-      <origin rpy="0 1.5708 0"/>
+      <origin rpy="-1.5708 0 0"/>
       <material name="Black"/>
     </visual>
     <collision>
       <geometry>
-        <cylinder radius="${wheel_radius}" length="${wheel_width}"/>
+        <sphere radius="${wheel_radius}"/>
       </geometry>
       <origin rpy="0 1.5708 0"/>
@@ -147,5 +151,5 @@
     <parent link="${prefix}base_link"/>
     <child link="${prefix}front_left_caster"/>
-    <origin xyz="${front_x} ${left_y} ${-base_height/2}"/>
+    <origin xyz="${front_x} ${left_y} ${-base_height/2 + caster_radius}"/>
   </joint>
   <!-- ========================= -->
@@ -181,5 +185,5 @@
     <parent link="${prefix}base_link"/>
     <child link="${prefix}front_right_caster"/>
-    <origin xyz="${front_x} ${right_y} ${-base_height/2}"/>
+    <origin xyz="${front_x} ${right_y} ${-base_height/2 + caster_radius}"/>
   </joint>
   <!-- ========================= -->
@@ -189,5 +193,5 @@
     <visual>
       <geometry>
-        <cylinder radius="0.035" length="0.03"/>
+        <cylinder radius="0.035" length="0.01"/>
       </geometry>
       <origin rpy="0 0 0"/>
@@ -196,11 +200,11 @@
     <collision>
       <geometry>
-        <cylinder radius="0.035" length="0.03"/>
-      </geometry>
-    </collision>
-    <inertial>
-      <mass value="0.1"/>
-      <inertia ixx="0.0001" iyy="0.0001" izz="0.0001"
-               ixy="0.0" ixz="0.0" iyz="0.0"/>
+        <cylinder radius="0.035" length="0.01"/>
+      </geometry>
+    </collision>
+    <inertial>
+      <mass value="1e-6"/>
+      <inertia ixx="1e-6" iyy="1e-6" izz="1e-6"
+               ixy="0.0" ixz="0.0" iyz="0.0"/>   <!--0.0001-->
     </inertial>
   </link>
@@ -208,21 +212,21 @@
     <parent link="${prefix}base_link"/>
     <child link="${prefix}lidar_link"/>
-    <origin xyz="0 0 ${base_height/2 + 0.02}"/>
+    <origin xyz="0 0 ${base_height/2 + 0.03}"/> <!--${base_height/2 + 0.02}-->
   </joint>
   <gazebo reference="${prefix}lidar_link">
-    <sensor type="gpu_lidar" name="lidar">
-      <topic>scan</topic>
+    <sensor name="lidar" type="gpu_lidar" >
+      <update_rate>10</update_rate>
+      <topic>/${ns}/scan</topic>
       <frame_id>${prefix}lidar_link</frame_id>
-      <update_rate>10</update_rate>
-      <ray>
+      <lidar>
         <scan>
           <horizontal>
             <samples>360</samples>
-            <min_angle>-3.14159</min_angle>
-            <max_angle>3.14159</max_angle>
+            <min_angle>-3.14</min_angle>
+            <max_angle>3.14</max_angle>
           </horizontal>
         </scan>
         <range>
-          <min>0.12</min>
+          <min>0.01</min>
           <max>8.0</max>
           <resolution>0.01</resolution>
@@ -231,7 +235,7 @@
           <type>gaussian</type>
           <mean>0.0</mean>
-          <stddev>0.01</stddev>
+          <stddev>0.001</stddev>
         </noise>
-      </ray>
+      </lidar>
       <always_on>1</always_on>
       <visualize>true</visualize>
@@ -255,5 +259,5 @@
   <gazebo reference="${prefix}imu_link">
     <sensor type="imu" name="imu">
-      <topic>imu</topic>
+      <topic>/${ns}/imu</topic>
       <frame_id>${prefix}imu_link</frame_id>
       <update_rate>100</update_rate>
@@ -267,10 +271,11 @@
     <plugin filename="gz-sim-diff-drive-system"
             name="gz::sim::systems::DiffDrive">
+            <render_engine>ogre2</render_engine>
       <left_joint>${prefix}left_wheel_joint</left_joint>
       <right_joint>${prefix}right_wheel_joint</right_joint>
       <wheel_separation>${base_width}</wheel_separation>
       <wheel_radius>${wheel_radius}</wheel_radius>
-      <topic>cmd_vel</topic>
-      <odom_topic>odom</odom_topic>
+      <topic>/${ns}/cmd_vel</topic>
+      <odom_topic>/${ns}/odom</odom_topic>
       <odom_frame>odom</odom_frame>
       <robot_base_frame>${prefix}base_link</robot_base_frame>
